File: power.kicad_sch (KiCad schematic)
At the start: 0 parts

Commit message: WIP: Power supply
Parts:
- added C1, C10, C11, C2: 22u, symbol Device:C
- added C12, C14, C3, C5, C9: 100n, symbol Device:C
- added C13, C4, C8: 10u, symbol Device:C
- added C15: 100u, SOP65P640X120-17N, symbol Device:C_Polarized
- added C6: 1u, symbol Device:C
- added C7: 100u, symbol Device:C
- added FB1: FerriteBead, symbol Device:FerriteBead
- added L1: 1.5u, symbol Device:L
- added L2: 2.2u, symbol Device:L
- added R1, R7: 30.1k, symbol Device:R
- added R2, R5, R8: 22.1k, symbol Device:R
- added R3: 100k, symbol Device:R
- added R4: 73.2k, symbol Device:R
- added R6: 1, symbol Device:R
- added U1: TPS54325PWP, Package_SO:Texas_HTSSOP-14-1EP_4.4x5mm_P0.65mm_EP3.4x5mm_Mask2.94x3.34mm_ThermalVias, symbol symbol_library:TPS54325PWP
- added U2: TPS54294PWP, SOP65P640X120-17N, symbol symbol_library:TPS54294PWP
Connections:
- new net: R7.2, R8.1, U1.2 (VFB)
- new net: C3.1, U2.2 (VBST1)
- new net: C3.2, L1.2, U2.3 (SW1)
- new net: R7.1, U1.1 (VO)
- new net: C12.1, U1.4 (SS)
- new net: R4.2, R5.1, U2.10 (VFB2)
- new net: R3.2, U2.12 (EN2), U2.6 (PG1)
- new net: C7.2, L2.1, U2.14 (SW2)
- new net: C7.1, U2.15 (VBST2)
- new net: R1.2, R2.1, U2.7 (VFB1)
- new net: C6.1, R3.1, U2.9 (VREG5)
- new net: FB1.2, R6.1
- new net +1V8: C1.1, C2.1, L1.1, R1.1
- new net +3.3V: C10.1, C11.1, FB1.1, L2.2, R4.1
- new net +3.3VA: R6.2
- new net GND: C1.2, C10.2, C11.2, C12.2, C13.2, C14.2, C15.2, C2.2, C4.2, C5.2, C6.2, C8.2, C9.2, R2.2, R5.2, R8.2, U1.15 (PwPd), U1.5 (GND), U2.13 (PGND2), U2.17 (PwPd), U2.4 (PGND1), U2.8 (GND)
- new net POWER_IN: C13.1, C14.1, C15.1, C4.1, C5.1, C8.1, C9.1, U1.13 (VIN), U1.14 (VCC), U1.7 (EN), U2.1 (VIN1), U2.16 (VIN2)
- no-connect marks 0 -> 1
Other:
- note added: "4.5V - 18V"
- note added: "Ip>2.8A, Irms>2.1A"
- note added: "Ip>2.9A, Irms>2.1A"
- title: (none) -> Power

Commit message: Finish power supply?
Parts:
- added C16: 10u, symbol Device:C
- added C17: 100n, symbol Device:C
- added C18, C19: 22u, symbol Device:C
- added L3: 2.2u, symbol Device:L
- added R9: 100k, symbol Device:R
Connections:
- net GND: now also U1.8 (PGND1), U1.9 (PGND2), C16.2, C18.2, C19.2
- net +1V0: now reaches R7.1, U1.1 (VO)
- net +1V0: now also C18.1, C19.1, L3.2
- net at U1.10 (SW1): now also U1.11 (SW2), C17.2, L3.1
- net at U1.12 (VBST): now also C17.1
- net at U1.3 (VREG5): now also C16.1, R9.1
- net at U1.6 (PG): now also U2.5 (EN1), R9.2
Other:
- note added: "Ip>3.5A, Irms>3.1A"
- moved on the sheet: C10, C11, FB1, L2, R4, R5, R6
